File: Power_Rail.kicad_sch (KiCad schematic)
At the start: 16 parts, among them J2 USB_C_Receptacle_USB2.0_16P, U3 AMS1117

Commit message: Schematic Clean Up
Other:
- moved on the sheet: C20, C21, C22, D4, R11, R12, U3

Commit message: PCB Update
Parts:
- J2: footprint Connector_USB:USB_C_Receptacle_GCT_USB4105-xx-A_16P_TopMnt_Horizontal -> Connector_USB:USB_C_Receptacle_HRO_TYPE-C-31-M-12
Changed lines of the file:
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@@
 			)
 		)
-		(property "Footprint" "Connector_USB:USB_C_Receptacle_GCT_USB4105-xx-A_16P_TopMnt_Horizontal"
+		(property "Footprint" "Connector_USB:USB_C_Receptacle_HRO_TYPE-C-31-M-12"
 			(at 97.79 45.72 0)
 			(effects

Commit message: Layout Update
Parts:
- added C42: 1uF, Capacitor_SMD:C_0603_1608Metric_Pad1.08x0.95mm_HandSolder, symbol Device:C
- added D26: PESD5V0U1BB_115, KSZ_KiCad_Footprint_Library:DIO_PESD5V0U1BB_115, symbol KSZ_KiCad_Symbol_Library:PESD5V0U1BB_115
Connections:
- net +5V: now also C42.1, D26.K2
- net GND: now also C42.2, D26.K1
Other:
- moved on the sheet: C19, D1, D2, D3, J2, R10, R7, R8, R9
