File: RP2040_Macropad_3x3.kicad_pcb (KiCad board)
At the start: 2 copper layers, 3.4 x 3 mm, 129 parts, among them IC1 W25Q16JVSNIQ, J1 Conn_01x03_Pin, J2 USB_C_Receptacle_USB2.0_16P, U1 RP2040, U10 MX1A-11NN, U11 MX1A-11NN, U12 MX1A-11NN, U13 MX1A-11NN, U2 SSD1306_128x32, U3 AMS1117, U4 MX1A-11NN, U5 MX1A-11NN, U6 MX1A-11NN, U7 SN74LVC1G17DCKR, U8 MX1A-11NN, U9 MX1A-11NN, Y1 ABM8-272-T3 12MHz

Commit message: PCB Update
Parts:
- J2: footprint Connector_USB:USB_C_Receptacle_GCT_USB4105-xx-A_16P_TopMnt_Horizontal -> Connector_USB:USB_C_Receptacle_HRO_TYPE-C-31-M-12; moved to B.Cu
- S10, S11, S3, S4, S5, S6, S7, S8, S9: moved to B.Cu
- moved C10 186.9 mm to (-76.8, 68.1)
- moved C11 186.9 mm to (-76.8, 70.6)
- moved C12 186.9 mm to (-76.8, 73.1)
- moved C13 186.9 mm to (-76.8, 75.6)
- moved C14 186.9 mm to (-76.8, 78.1)
- moved C15 186.9 mm to (-76.8, 80.6)
- moved C16 186.9 mm to (-76.8, 83.1)
- moved C17 186.9 mm to (-76.8, 85.6)
- moved C18 186.9 mm to (-72.5, 68.1)
- moved C19 186.9 mm to (-53.4, 68.1)
- moved C2 186.9 mm to (-81.2, 68.1)
- moved C20 186.9 mm to (-53.4, 70.6)
- moved C21 186.9 mm to (-53.4, 73.1)
- moved C22 186.9 mm to (-53.4, 75.6)
- moved C23 186.9 mm to (-112.4, 48.5)
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Other:
- board size 3.4 x 3 mm -> 73.7 x 109.8 mm

Commit message: Layout Update
Parts:
- added C42: 1uF, Capacitor_SMD:C_0603_1608Metric_Pad1.08x0.95mm_HandSolder, B.Cu at (122.8, 38.7)
- added D26: PESD5V0U1BB_115, KSZ_KiCad_Footprint_Library:DIO_PESD5V0U1BB_115, B.Cu at (123.3, 37.1)
- C1, C10, C11, C12, C13, C14, C15, C16, C17, C18, C19, C2, C20, C21, C23, C24, C25, C26, C27, C28, C29, C3, C30, C31, C32, C33, C34, C35, C36, C37, C38, C39, C4, C40, C41, C5, C6, C7, C8, C9, D1, D10, D11, D12, D13, D14, D15, D16, D17, D18, D19, D2, D20, D21, D22, D23, D24, D25, D3, D5, D6, D7, D8, D9, IC1, R1, R10, R13, R14, R15, R16, R17, R18, R19, R2, R20, R21, R22, R23, R24, R25, R26, R27, R28, R3, R4, R5, R6, R9, S1, S2, U1, U3, Y1: moved to B.Cu
- U7: value SN74LVC1G17DCKR -> SN74LV1T34DBVR; footprint KSZ_KiCad_Footprint_Library:SOT65P210X110-5N -> KSZ_KiCad_Footprint_Library:SOT95P280X145-5N; moved to B.Cu
- moved C23 292.5 mm to (172.1, 116.8), turned to 90 degrees
- moved C31 281.3 mm to (169.2, 98.6), turned to 180 degrees
- moved U1 277.4 mm to (153.4, 134.5), turned to -90 degrees
- moved C35 276.0 mm to (167.8, 50.9)
- moved C41 273.6 mm to (170.0, 57.3)
- moved C32 272.2 mm to (156.8, 116.1)
- moved C38 270.1 mm to (166.4, 57.3)
- moved R16 269.8 mm to (159.8, 125.9), turned to -90 degrees
- moved R15 268.7 mm to (158.1, 125.9), turned to -90 degrees
- moved R13 267.9 mm to (156.2, 125.9), turned to -90 degrees
- moved R14 266.6 mm to (156.4, 122.1), turned to 180 degrees
- moved C30 266.4 mm to (156.8, 78.1)
- moved U7 266.1 mm to (169.3, 117.3), turned to 90 degrees
- moved R19 265.8 mm to (166.4, 53.9), turned to 180 degrees
- moved C28 265.2 mm to (150.2, 98.7), turned to 180 degrees
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Connections:
- C3 pad 1: /VREG_OUT -> /VREG_VOUT
- C5 pad 1: /VREG_OUT -> /VREG_VOUT
- C7 pad 1: /VREG_OUT -> /VREG_VOUT
- D13 pad 2: Net-(D13-DOUT) -> unconnected-(D13-DOUT-Pad2)
- D13 pad 4: /Switch_Matrix/LED_ROW_0 -> Net-(D13-DIN)
- D15 pad 2: Net-(D15-DOUT) -> /Switch_Matrix/LED_ROW_1
- D15 pad 4: /Switch_Matrix/LED_ROW_2 -> Net-(D15-DIN)
- D20 pad 2: Net-(D20-DOUT) -> Net-(D13-DIN)
- D20 pad 4: Net-(D13-DOUT) -> Net-(D20-DIN)
- D22 pad 2: Net-(D22-DOUT) -> Net-(D15-DIN)
- D22 pad 4: Net-(D15-DOUT) -> Net-(D22-DIN)
- D23 pad 2: /Switch_Matrix/LED_ROW_1 -> Net-(D20-DIN)
- D23 pad 4: Net-(D20-DOUT) -> /Switch_Matrix/LED_ROW_2
- D25 pad 2: unconnected-(D25-DOUT-Pad2) -> Net-(D22-DIN)
- D25 pad 4: Net-(D22-DOUT) -> /Switch_Matrix/LED_ROW_0
- MT1 pad 1: /COL_0 -> /Switch_Matrix/COL_0_1
- MT2 pad 1: /COL_1 -> /Switch_Matrix/COL_1_1
- MT3 pad 1: /COL_2 -> /Switch_Matrix/COL_2_1
- R13 pad 1: /COL_0 -> /Switch_Matrix/COL_0_1
- R15 pad 1: /COL_1 -> /Switch_Matrix/COL_1_1
- R16 pad 1: /COL_2 -> /Switch_Matrix/COL_2_1
- R5 pad 1: +3.3V -> +3V3
- R5 pad 2: /I2C0_SDA -> /I2C1_SDA
- R6 pad 1: /I2C0_SCL -> +3V3
- R6 pad 2: +3.3V -> /I2C1_SCL
- S10 pad 1: /COL_2 -> /Switch_Matrix/COL_2_1
- S11 pad 1: /COL_2 -> /Switch_Matrix/COL_2_1
- S3 pad 1: /COL_0 -> /Switch_Matrix/COL_0_1
- S4 pad 1: /COL_0 -> /Switch_Matrix/COL_0_1
- S5 pad 1: /COL_0 -> /Switch_Matrix/COL_0_1
- S6 pad 1: /COL_1 -> /Switch_Matrix/COL_1_1
- S7 pad 1: /COL_1 -> /Switch_Matrix/COL_1_1
- S8 pad 1: /COL_1 -> /Switch_Matrix/COL_1_1
- S9 pad 1: /COL_2 -> /Switch_Matrix/COL_2_1
- U1 pad 2: /ROW_0 -> /ROW_3
- U1 pad 3: /ROW_1 -> /ROW_0
- U1 pad 36: /LED_BUFFER -> unconnected-(U1-GPIO24-Pad36)
- U1 pad 39: unconnected-(U1-GPIO27/ADC1-Pad39) -> /I2C1_SCL
- U1 pad 4: /ROW_2 -> /ROW_1
- U1 pad 40: unconnected-(U1-GPIO28/ADC2-Pad40) -> /I2C1_SDA
- U1 pad 45: /VREG_OUT -> /VREG_VOUT
- U1 pad 5: /ROW_3 -> /ROW_2
- U1 pad 6: /I2C0_SDA -> unconnected-(U1-GPIO4-Pad6)
- U1 pad 7: /I2C0_SCL -> /LED_BUFFER
- U2 pad 3: /I2C0_SCL -> /I2C1_SCL
- U2 pad 4: /I2C0_SDA -> /I2C1_SDA
Routing:
- net +3V3: track 0.00 -> 350.5 mm, vias 0 -> 10
- net +5V_LED: track 0.00 -> 312.1 mm, vias 0 -> 3
- net /ROW_3: track 0.00 -> 190.9 mm, vias 0 -> 2
- net +5V: track 0.00 -> 185.4 mm, vias 0 -> 8
- net /ROW_0: track 0.00 -> 165.1 mm
- net /ENC0_A: track 0.00 -> 155.0 mm
- net /ENC0_B: track 0.00 -> 151.3 mm, vias 0 -> 2
- net /ROW_1: track 0.00 -> 145.9 mm
- net /Power_Rail/USB_CON_N: track 0.00 -> 145.5 mm, vias 0 -> 1
- net /Power_Rail/USB_CON_P: track 0.00 -> 143.6 mm, vias 0 -> 1
- net /ENC1_A: track 0.00 -> 139.3 mm, vias 0 -> 2
- net /ENC1_B: track 0.00 -> 131.7 mm, vias 0 -> 2
- net /Switch_Matrix/COL_0_1: track 0.00 -> 125.5 mm, vias 0 -> 4
- net /ROW_2: track 0.00 -> 125.4 mm
- net /ENC2_A: track 0.00 -> 120.0 mm, vias 0 -> 2
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- added copper zone on B.Cu, net +3V3
- added copper zone on B.Cu, net +5V
- added copper zone on F.Cu, net +5V
- added copper zone on F.Cu, net +5V_LED
- added copper zone on B.Cu, net GND
- added copper zone on In1.Cu, net GND
- added copper zone on In2.Cu, net GND
Other:
- board size 73.7 x 109.8 mm -> 73.7 x 121.5 mm
- copper layers 2 -> 4
