File: RP2040_Macropad_3x3.kicad_sch (KiCad schematic)
At the start: 17 parts

Commit message: USB, FLASH & Power Rail Update
Parts:
- added C? (x2): 22uF, Capacitor_SMD:C_0603_1608Metric_Pad1.08x0.95mm_HandSolder, symbol Device:C
- added C?: 100nF, Capacitor_SMD:C_0603_1608Metric_Pad1.08x0.95mm_HandSolder, symbol Device:C
- added C?: 2.2uF, Capacitor_SMD:C_0603_1608Metric_Pad1.08x0.95mm_HandSolder, symbol Device:C
- added C?: 1uF, Capacitor_SMD:C_0603_1608Metric_Pad1.08x0.95mm_HandSolder, symbol Device:C
- added D? (x3): PESD5V0U1BB_115, KSZ_KiCad_Footprint_Library:DIO_PESD5V0U1BB_115, symbol KSZ_KiCad_Symbol_Library:PESD5V0U1BB_115
- added IC?: W25Q16JVSNIQ, KSZ_KiCad_Footprint_Library:SOIC127P600X175-8N, symbol KSZ_KiCad_Symbol_Library:W25Q16JVSNIQ
- added J?: USB_C_Receptacle_USB2.0_16P, symbol Connector:USB_C_Receptacle_USB2.0_16P
- added R? (x2): 27, Resistor_SMD:R_0603_1608Metric_Pad0.98x0.95mm_HandSolder, symbol Device:R
- added R?: 200, Resistor_SMD:R_0603_1608Metric_Pad0.98x0.95mm_HandSolder, symbol Device:R
- added R? (x2): 5.1k, Resistor_SMD:R_0603_1608Metric_Pad0.98x0.95mm_HandSolder, symbol Device:R
- added U?: AMS1117, KSZ_KiCad_Footprint_Library:SOT229P700X180-4N, symbol KSZ_KiCad_Symbol_Library:AMS1117
- C? (x2): value 1uF -> 2.2uF
- C?: value 100nF -> 2.2uF
Connections:
- net +3V3: now also C?.1, C?.1, C?.1, IC?.8 (VCC), R?.2, U?.2 (VOUT), U?.4 (VOUT); no longer C?.1, U?.43 (ADC_AVDD)
- net GND: now also U?.19 (TESTEN), U?.57 (GND), C?.2, C?.2, C?.2, C?.2, C?.2, D?.K1, D?.K1, D?.K1, IC?.4 (GND), J?.A1 (GND), J?.A12 (GND), J?.B1 (GND), J?.B12 (GND), J?.S1 (SHIELD), R?.2, R?.2, U?.1 (ADJ/GND)
- net VREG_OUT: no longer C?.1, C?.1, C?.1, U?.23 (DVDD), U?.50 (DVDD)
- net USB_N: now reaches U?.46 (USB_DM)
- net USB_N: now also R?.1
- net USB_P: now reaches U?.47 (USB_DP)
- net USB_P: now also R?.1
- net QSPI_SD3: now reaches U?.51 (QSPI_SD3)
- net QSPI_SD3: now also IC?.7 (~{HOLD_OR_}~{RESET_}(IO3))
- net QSPI_SCLK: now reaches U?.52 (QSPI_SCLK)
- net QSPI_SCLK: now also IC?.6 (CLK)
- net QSPI_SD0: now reaches U?.53 (QSPI_SD0)
- net QSPI_SD0: now also IC?.5 (DI_(IO0))
- net QSPI_SD2: now reaches U?.54 (QSPI_SD2)
- net QSPI_SD2: now also IC?.3 (~{WP_}(IO2))
- net QSPI_SD1: now reaches U?.55 (QSPI_SD1)
- net QSPI_SD1: now also IC?.2 (DO_(IO1))
- net QSPI_CSN: now reaches U?.56 (QSPI_CSN)
- net QSPI_CSN: now also IC?.1 (~{CS})
- new net: J?.A5 (CC1), R?.1
- new net: J?.B5 (CC2), R?.1
- new net +5V: C?.1, C?.1, D?.K2, J?.A4 (VBUS), J?.A9 (VBUS), J?.B4 (VBUS), J?.B9 (VBUS), U?.3 (VIN)
- new net ADC_AVDD: C?.1, R?.1, U?.43 (ADC_AVDD)
- new net USB_CON_N: D?.K2, J?.A7 (D-), J?.B7 (D-), R?.2
- new net USB_CON_P: D?.K2, J?.A6 (D+), J?.B6 (D+), R?.2
- new net VREG_VOUT: C?.1, C?.1, C?.1, U?.23 (DVDD), U?.50 (DVDD)
- no-connect marks 0 -> 2
Other:
- note added: "DC-DC Converter 5V -> 3.3V"
- note added: "Flash"
- note added: "USB"
- moved on the sheet: C?

Commit message: Schematic Update
Parts:
- removed C? (x10): 100nF, Capacitor_SMD:C_0603_1608Metric_Pad1.08x0.95mm_HandSolder, symbol Device:C
- removed C? (x4): 2.2uF, Capacitor_SMD:C_0603_1608Metric_Pad1.08x0.95mm_HandSolder, symbol Device:C
- removed C? (x2): 22uF, Capacitor_SMD:C_0603_1608Metric_Pad1.08x0.95mm_HandSolder, symbol Device:C
- removed C?: 1uF, Capacitor_SMD:C_0603_1608Metric_Pad1.08x0.95mm_HandSolder, symbol Device:C
- removed C? (x2): 15pF, Capacitor_SMD:C_0603_1608Metric_Pad1.08x0.95mm_HandSolder, symbol Device:C
- removed D? (x3): PESD5V0U1BB_115, KSZ_KiCad_Footprint_Library:DIO_PESD5V0U1BB_115, symbol KSZ_KiCad_Symbol_Library:PESD5V0U1BB_115
- removed IC?: W25Q16JVSNIQ, KSZ_KiCad_Footprint_Library:SOIC127P600X175-8N, symbol KSZ_KiCad_Symbol_Library:W25Q16JVSNIQ
- removed J?: USB_C_Receptacle_USB2.0_16P, symbol Connector:USB_C_Receptacle_USB2.0_16P
- removed R? (x2): 27, Resistor_SMD:R_0603_1608Metric_Pad0.98x0.95mm_HandSolder, symbol Device:R
- removed R?: 200, Resistor_SMD:R_0603_1608Metric_Pad0.98x0.95mm_HandSolder, symbol Device:R
- removed R? (x2): 5.1k, Resistor_SMD:R_0603_1608Metric_Pad0.98x0.95mm_HandSolder, symbol Device:R
- removed R?: 1k, Resistor_SMD:R_0603_1608Metric_Pad0.98x0.95mm_HandSolder, symbol Device:R
- removed U?: AMS1117, KSZ_KiCad_Footprint_Library:SOT229P700X180-4N, symbol KSZ_KiCad_Symbol_Library:AMS1117
- removed Y?: ABM8-272-T3 12MHz, Crystal:Crystal_SMD_3225-4Pin_3.2x2.5mm_HandSoldering, symbol Device:Crystal_GND24
- added C1: 100nF, Capacitor_SMD:C_0603_1608Metric_Pad1.08x0.95mm_HandSolder, symbol Device:C
- added H1, H2, H3, H4: MountingHole_Pad, MountingHole:MountingHole_3.2mm_M3_Pad, symbol Mechanical:MountingHole_Pad
- added U2: SSD1306_128x32, KSZ_KiCad_Footprint_Library:SSD1306_128x32_Display_Module, symbol KSZ_KiCad_Symbol_Library:SSD1306_128x32_Display_Module
- gave numbers to parts that had none: 1
Connections:
- net +3V3: now also C1.2, U2.2 (VDD); no longer U1.1 (IOVDD), U1.10 (IOVDD), U1.22 (IOVDD), U1.33 (IOVDD), U1.42 (IOVDD), U1.44 (VREG_VIN), U1.48 (USB_VDD), U1.49 (IOVDD)
- net GND: now also C1.1, H1.1, H2.1, H3.1, H4.1, U2.1 (GND)
- net COL_0: now reaches U1.13 (GPIO10)
- net COL_1: now reaches U1.14 (GPIO11)
- net COL_2: now reaches U1.15 (GPIO12)
- net ENC0_A: now reaches U1.18 (GPIO15)
- net ROW_0: now reaches U1.2 (GPIO0)
- net SWCLK: now reaches U1.24 (SWCLK)
- net SWD: now reaches U1.25 (SWD)
- net RUN: now reaches U1.26 (RUN)
- net ENC0_B: now reaches U1.27 (GPIO16)
- net ENC1_A: now reaches U1.28 (GPIO17)
- net ENC1_B: now reaches U1.29 (GPIO18)
- net ROW_1: now reaches U1.3 (GPIO1)
- net ENC2_A: now reaches U1.30 (GPIO19)
- net ENC2_B: now reaches U1.31 (GPIO20)
- net LED_BUFFER: now reaches U1.36 (GPIO24)
- net ROW_2: now reaches U1.4 (GPIO2)
- net ROW_3: now reaches U1.5 (GPIO3)
- net I2C0_SDA: now reaches U1.6 (GPIO4)
- net I2C0_SDA: now also U2.4 (SDA)
- net I2C0_SCL: now reaches U1.7 (GPIO5)
- net I2C0_SCL: now also U2.3 (SCK)
- new net IOVDD: U1.1 (IOVDD), U1.10 (IOVDD), U1.22 (IOVDD), U1.33 (IOVDD), U1.42 (IOVDD), U1.49 (IOVDD)
- new net USB_VDD: U1.48 (USB_VDD)
- new net VREG_VIN: U1.44 (VREG_VIN)
- no-connect marks 2 -> 14
Other:
- added sheet Power_Rail (Power_Rail.kicad_sch)
- added sheet RP2040_External_Peripherals (RP2040_External_Peripherals.kicad_sch)
- added sheet Switch_Matrix (Switch_Matrix.kicad_sch)
- note removed: "Crystal oscillator"
- note removed: "DC-DC Converter 5V -> 3.3V"
- note removed: "Decoupling capacitors"
- note removed: "Flash"
- note removed: "USB"

Commit message: Schematic Clean Up
Other:
- note added: "External Peripherals"
- note added: "Mounting Holes"
- note added: "OLED Display"
- note added: "Power Rail"
- note added: "Switch Matrix"
- moved on the sheet: C1, H1, H2, H3, H4, U2

Commit message: Layout Update
Connections:
- net VREG_OUT is gone; now on net VREG_VOUT: U1.45 (VREG_VOUT)
- net LED_BUFFER: now also U1.7 (GPIO5); no longer U1.36 (GPIO24)
- net ROW_0: now also U1.3 (GPIO1); no longer U1.2 (GPIO0)
- net ROW_1: now also U1.4 (GPIO2); no longer U1.3 (GPIO1)
- net ROW_2: now also U1.5 (GPIO3); no longer U1.4 (GPIO2)
- net ROW_3: now also U1.2 (GPIO0); no longer U1.5 (GPIO3)
- net I2C1_SCL: now reaches U1.39 (GPIO27/ADC1)
- net I2C1_SCL: now also U2.3 (SCK)
- net I2C1_SDA: now reaches U1.40 (GPIO28/ADC2)
- net I2C1_SDA: now also U2.4 (SDA)
- removed net I2C0_SCL: U1.7 (GPIO5), U2.3 (SCK)
- net I2C0_SDA: no longer names the net of U1.6 (GPIO4)
- net I2C0_SDA: no longer U2.4 (SDA)
Other:
- sheet RP2040_External_Peripherals ports: added I2C1_SCL, I2C1_SDA; removed I2C0_SCL, I2C0_SDA
Changed lines of the file:
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@@
 	)
 	(no_connect
+		(at 78.74 102.87)
+	)
+	(no_connect
 		(at 78.74 95.25)
 	)
@@
 	)
 	(no_connect
-		(at 78.74 113.03)
+		(at 33.02 90.17)
 	)
 	(no_connect
@@
 	)
 	(no_connect
-		(at 78.74 110.49)
-	)
-	(no_connect
 		(at 78.74 105.41)
 	)
@@
 	(wire
 		(pts
-			(xy 24.13 92.71) (xy 33.02 92.71)
-		)
-		(stroke
-			(width 0)
-			(type default)
-		)
-	)
-	(wire
-		(pts
 			(xy 119.38 43.18) (xy 119.38 49.53)
 		)
@@
 	(wire
 		(pts
-			(xy 78.74 125.73) (xy 81.28 125.73)
+			(xy 87.63 110.49) (xy 78.74 110.49)
 		)
 		(stroke
@@
 	(wire
 		(pts
-			(xy 78.74 54.61) (xy 87.63 54.61)
+			(xy 78.74 125.73) (xy 81.28 125.73)
 		)
 		(stroke
@@
 	(wire
 		(pts
-			(xy 24.13 90.17) (xy 33.02 90.17)
+			(xy 78.74 54.61) (xy 87.63 54.61)
 		)
 		(stroke
@@
 	(wire
 		(pts
-			(xy 78.74 102.87) (xy 91.44 102.87)
+			(xy 33.02 92.71) (xy 20.32 92.71)
 		)
 		(stroke
@@
 	(wire
 		(pts
+			(xy 87.63 113.03) (xy 78.74 113.03)
+		)
+		(stroke
+			(width 0)
+			(type default)
+		)
+	)
+	(wire
+		(pts
 			(xy 167.64 57.15) (xy 179.07 57.15)
 		)
@@
 		)
 	)
-	(label "I2C0_SDA"
-		(at 24.13 90.17 0)
-		(effects
-			(font
-				(size 1.27 1.27)
-			)
-			(justify left bottom)
-		)
-	)
 	(label "ENC0_A"
 		(at 87.63 80.01 180)
@@
 		)
 	)
-	(label "I2C0_SCL"
+	(label "I2C1_SCL"
 		(at 144.78 43.18 180)
 		(effects
@@
 		)
 	)
+	(label "I2C1_SCL"
+		(at 87.63 110.49 180)
+		(effects
+			(font
+				(size 1.27 1.27)
+			)
+			(justify right bottom)
+		)
+	)
 	(label "IOVDD"
 		(at 87.63 41.91 180)
@@
 	)
 	(label "ROW_1"
-		(at 24.13 82.55 0)
+		(at 24.13 85.09 0)
 		(effects
 			(font
@@
 		)
 	)
+	(label "I2C1_SDA"
+		(at 87.63 113.03 180)
+		(effects
+			(font
+				(size 1.27 1.27)
+			)
+			(justify right bottom)
+		)
+	)
 	(label "ENC2_A"
 		(at 87.63 90.17 180)
@@
 		)
 	)
-	(label "I2C0_SDA"
+	(label "I2C1_SDA"
 		(at 167.64 69.85 0)
 		(effects
@@
 		)
 	)
-	(label "VREG_OUT"
+	(label "VREG_VOUT"
 		(at 87.63 49.53 180)
 		(effects
@@
 	)
 	(label "ROW_3"
-		(at 24.13 87.63 0)
+		(at 24.13 80.01 0)
 		(effects
 			(font
@@
 	)
 	(label "LED_BUFFER"
-		(at 91.44 102.87 180)
+		(at 20.32 92.71 0)
 		(effects
 			(font
 				(size 1.27 1.27)
 			)
-			(justify right bottom)
+			(justify left bottom)
 		)
 	)
@@
 	)
 	(label "ROW_2"
-		(at 24.13 85.09 0)
+		(at 24.13 87.63 0)
 		(effects
 			(font
@@
 		)
 	)
-	(label "VREG_OUT"
+	(label "VREG_VOUT"
 		(at 167.64 36.83 0)
 		(effects
@@
 		)
 	)
-	(label "I2C0_SCL"
+	(label "I2C1_SCL"
 		(at 167.64 72.39 0)
 		(effects
@@
 	)
 	(label "ROW_0"
-		(at 24.13 80.01 0)
+		(at 24.13 82.55 0)
 		(effects
 			(font
@@
 		)
 	)
-	(label "I2C0_SCL"
-		(at 24.13 92.71 0)
-		(effects
-			(font
-				(size 1.27 1.27)
-			)
-			(justify left bottom)
-		)
-	)
 	(label "ENC1_B"
 		(at 87.63 87.63 180)
@@
 		)
 	)
-	(label "I2C0_SDA"
+	(label "I2C1_SDA"
 		(at 144.78 39.37 180)
 		(effects
@@
 			)
 		)
-		(pin "I2C0_SDA" input
-			(at 179.07 69.85 180)
+		(pin "I2C1_SCL" input
+			(at 179.07 72.39 180)
 			(effects
 				(font
@@
 			)
 		)
-		(pin "I2C0_SCL" input
-			(at 179.07 72.39 180)
+		(pin "I2C1_SDA" input
+			(at 179.07 69.85 180)
 			(effects
 				(font
