File: Switch_Matrix.kicad_sch (KiCad schematic)
At the start: 78 parts, among them U10 MX1A-11NN, U11 MX1A-11NN, U12 MX1A-11NN, U13 MX1A-11NN, U4 MX1A-11NN, U5 MX1A-11NN, U6 MX1A-11NN, U7 SN74LVC1G17DCKR, U8 MX1A-11NN, U9 MX1A-11NN

Commit message: Schematic Clean Up
Other:
- note added: "Encoders"
- note added: "LED Matrix"
- note added: "Logic Level Converter 3.3V -> 5V"
- note added: "Switch Matrix"
- moved on the sheet: C23, C24, C25, C26, C27, C28, C29, C30, C31, C32, C33, C34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

Commit message: Layout Update
Parts:
- removed U7: SN74LVC1G17DCKR, KSZ_KiCad_Footprint_Library:SOT65P210X110-5N, symbol KSZ_KiCad_Symbol_Library:SN74LVC1G17DCKR
- added U7: SN74LV1T34DBVR, KSZ_KiCad_Footprint_Library:SOT95P280X145-5N, symbol KSZ_KiCad_Symbol_Library:SN74LV1T34DBVR
Connections:
- net +5V: now also U7.5 (VCC)
- net COL_0: no longer MT1.1, R13.1, S3.1, S4.1, S5.1
- net COL_1: no longer MT2.1, R15.1, S6.1, S7.1, S8.1
- net COL_2: no longer MT3.1, R16.1, S10.1, S11.1, S9.1
- net GND: now also U7.1 (NC), U7.3 (GND)
- net LED_ROW_0: now also D25.4 (DIN), U7.4 (Y); no longer D13.4 (DIN)
- net LED_ROW_1: now also D15.2 (DOUT); no longer D23.2 (DOUT)
- net LED_ROW_2: now also D23.4 (DIN); no longer D15.4 (DIN)
- net at R14.1: now also U7.2 (A)
- net at D20.2 (DOUT): now also D13.4 (DIN); no longer D23.4 (DIN)
- net at D25.2 (DOUT): now also D22.4 (DIN)
- net at D22.2 (DOUT): now also D15.4 (DIN); no longer D25.4 (DIN)
- net at D20.4 (DIN): now also D23.2 (DOUT); no longer D13.2 (DOUT)
- new net COL_0_1: MT1.1, R13.1, S3.1, S4.1, S5.1
- new net COL_1_1: MT2.1, R15.1, S6.1, S7.1, S8.1
- new net COL_2_1: MT3.1, R16.1, S10.1, S11.1, S9.1
Other:
- moved on the sheet: C23, D13, D15, D20, D22, D23, D25, R14
